File: hardware/linefollower.sch (EAGLE design)
At the start: 27 parts, among them IC1 LD117AV, IC2 LD117AV

Commit message: quick fix; added 1 sensor
Parts:
- added R17: 200, resistor:R-EU_0204/5
- added R18: 10k, resistor:R-EU_0204/5
- added R19: 910, resistor:R-EU_0204/5
- added R20: 470, resistor:R-EU_0204/5
- added U$6: CNY70, cny70:CNY70
Connections:
- removed net S4: R15.1, R16.1, R16.2, R8.1, U$5.EMI
- new net GND1: R17.1
- new net N$5: R17.2, U$6.C
- new net S5: R15.1, R16.1, R16.2, R18.1, R19.1, R20.1, R20.2, R8.1, U$5.EMI, U$6.EMI
- net +5V: now also U$6.A, U$6.COL
- net GND: now also R18.2, R19.2
Other:
- moved on the sheet: R15, R16, R4, R8, U$5

Commit message: added driver circuit, renumbered parts
Parts:
- removed U$1: (no value), BluePill:BLUE_PILL
- added ST1: (no value), BluePill:BLUE_PILL
- added TB66121: TB6612FNG, TB6612FNG:TB6612FNG
- C2: value 10uF -> 100nF
- C3: value 100nF -> 10uF
- R12, R14, R16, R20: value 470 -> 10k
- R17: value 200 -> 910
- R5: value 10k -> 200
- R6, R7, R8: value 10k -> 470
- R9: value 910 -> 470
- renumbered U$2 to PC1, U$3 to PC2, U$4 to PC3, U$5 to PC5, U$6 to PC4
Connections:
- new net A_IN_1: ST1.PB3, TB66121.AIN1
- new net A_IN_2: ST1.PB4, TB66121.AIN2
- new net A_OUT_1: TB66121.A1
- new net A_OUT_2: TB66121.A2
- new net B_IN_1: ST1.PB5, TB66121.BIN1
- new net B_IN_2: ST1.PB6, TB66121.BIN2
- new net B_OUT_1: TB66121.B1
- new net B_OUT_2: TB66121.B2
- new net PWM_A: ST1.PB0, TB66121.PWMA
- new net PWM_B: ST1.PB1, TB66121.PWMB
- new net S4: ST1.PA3
- new net STBY: TB66121.STBY
- net +12V: now also TB66121.VM; no longer C3.1, IC2.IN
- net +3V3: now also IC2.OUT, ST1.VBAT, TB66121.VCC; no longer IC1.OUT, U$1.VBAT
- net +5V: now also C3.1, IC1.OUT, IC2.IN; no longer IC2.OUT
- net GND: now also R12.2, R14.2, R16.2, R17.2, R20.2, R5.1, ST1.GND, TB66121.GND1, TB66121.GND2, TB66121.GND3; no longer R4.1, R5.2, R6.2, R7.2, R8.2, R9.2
- net GND1: now also R4.1; no longer R17.1
- net N$4: now also R5.2; no longer R4.2
- net N$5: now also R4.2; no longer R17.2
- net S1: now also R6.1, R6.2, ST1.PA0; no longer R12.2, R5.1
- net S2: now also R13.1, R14.1, R7.1, R7.2, ST1.PA1; no longer R10.1, R10.2, R6.1, R9.1
- net S3: now also R15.1, R16.1, R8.1, R8.2, ST1.PA2; no longer R13.1, R14.1, R14.2, R7.1
- net S5: now also R10.1, R10.2, R17.1, R9.1, R9.2, ST1.PA4; no longer R15.1, R16.1, R16.2, R20.2, R8.1
Other:
- note added: "MCU"
- note added: "STEROWNIK SILNIKÓW"
- moved on the sheet: C1, C2, C3, C4, IC1, IC2, R10, R12, R13, R14, R15, R16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

Commit message: updated schematic
Parts:
- added C5: 100nF, resistor:C-EU025-024X044
- added S1: TL32PO, switch:TL32PO
- R10, R6, R7, R8, R9: value 470 -> 330
- R11, R13, R15, R17, R19: value 910 -> 680
Connections:
- net +12V: now also C5.1, S1.O
- net GND: now also C5.2
Other:
- note added: "PRZEŁĄCZNIK"
- moved on the sheet: C1, C3, IC1

Commit message: added initial documentation and BOM, updated schematic
Parts:
- removed IC1: LD117AV, v-reg:LD117AV
- added IC3: 7805T, linear:7805T
- R1, R2, R3, R4, R5: value 200 -> 150
Connections:
- net +12V: now also IC3.VI; no longer IC1.IN
- net +5V: now also IC3.VO; no longer IC1.OUT
- net A_IN_1: now also ST1.PB6; no longer ST1.PB3
- net A_IN_2: now also ST1.PB5; no longer ST1.PB4
- net B_IN_1: now also ST1.PB8; no longer ST1.PB5
- net B_IN_2: now also ST1.PB9; no longer ST1.PB6
- net GND: now also IC3.GND; no longer IC1.ADJ
- net STBY: now also ST1.PB7
